File: Buck-Boost/control/control_board.kicad_pcb (KiCad board)
At the start: 4 copper layers, 104 x 33 mm, 66 parts, among them IC1 F2800137RGZR, J1 Conn_01x05_Header, J8 Conn_01x02_Pin, J9 Conn_02x04_Counter_Clockwise, U1 LMV321, U10 LMV321, U2 TPS562202, U6 IR2101, U7 TCAN3414DR, U8 LD1117S12TR_SOT223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

Commit message: buck-boost/control & buck-boost/variant1 - corrected the pin-config
Parts:
- added R15: 100K, >=62.5mW, 0402, Resistor_SMD:R_0805_2012Metric, B.Cu at (165.7, 80.5)
- R10: value 453K, >=62.5mW, 0402 -> 732K, >=62.5mW, 0402
- R11: value 49.9K, >=62.5mW, 0402 -> 101K, >=62.5mW, 0402
- R5: value 10K, >=62.5mW, 0402 -> 16.9K, >=62.5mW, 0402
- moved C14 0.71 mm to (135.1, 65.0), turned to 0 degrees
Connections:
- net /Iin renamed /I_hv
- net /Iout renamed /I_lv
- net Iin_+ renamed I_hv_+
- net Iin_- renamed I_hv_-
- net Iout_+ renamed I_lv_+
- net Iout_- renamed I_lv_-
- C11 pad 1: +3.3V -> +1.2V
- C12 pad 1: +3.3V -> +1.2V
- C13 pad 1: +3.3V -> +1.2V
- C15 pad 1: +1.2V -> +3.3V
- C16 pad 1: +1.2V -> +3.3V
- C17 pad 1: +1.2V -> +3.3V
- C18 pad 1: +1.2V -> +3.3V
- C2 pad 2: HV+ -> LV+
- C4 pad 2: HV+ -> LV+
- C9 pad 1: +3.3V -> +1.2V
- D1 pad 1: HV+ -> LV+
- IC1 pad 18: +1.2V -> +3.3V
- IC1 pad 34: +1.2V -> +3.3V
- IC1 pad 35: +3.3V -> +1.2V
- IC1 pad 44: +3.3V -> +1.2V
- IC1 pad 45: +1.2V -> +3.3V
- J1 pad 29: unconnected-(J1-Pin_29-Pad29) -> LV+
- PS1 pad 2: HV+ -> LV+
- PS1 pad 3: HV+ -> Net-(PS1-EN/UVLO)
- R5 pad 1: HV+ -> Net-(PS1-EN/UVLO)
Routing:
- net LV+: track 0.00 -> 72.7 mm
- net HV+: track 21.6 -> 0.00 mm
- net +1.2V: track 42.4 -> 29.0 mm, vias 4 -> 5
- net Net-(PS1-EN/UVLO): track 0.00 -> 3.45 mm
- net +3.3V: track 25.6 -> 25.7 mm, vias 19 -> 18
