File: Buck-Boost/variant1/power_board.kicad_sch (KiCad schematic)
At the start: 24 parts, among them J1 Conn_01x05_Header, Q1 NMOS, Vds>=80V, Rds<=1.5mOhm, Q2 NMOS, Vds>=80V, Rds<=1.5mOhm, Q3 NMOS, Vds>=80V, Rds<=1.5mOhm, Q4 NMOS, Vds>=80V, Rds<=1.5mOhm, Q5 NMOS, Vds>=80V, Rds<=1.5mOhm, Q6 NMOS, Vds>=80V, Rds<=1.5mOhm, Q7 NMOS, Vds>=80V, Rds<=1.5mOhm, Q8 NMOS, Vds>=80V, Rds<=1.5mOhm

Commit message: buck-boost/control & buck-boost/variant1 - corrected the pin-config
Parts:
- added C2: >22uF, >25V, Capacitor_SMD:C_0805_2012Metric, symbol Device:C_Small
- R18: value 1mOhm, >=3W -> 500uOhm, >=3W
Connections:
- net Iin_+: no longer J1.12 (Pin_12)
- net Iin_-: no longer J1.6 (Pin_6)
- net Iout_+: no longer J1.32 (Pin_32)
- net Iout_-: no longer J1.30 (Pin_30)
- net LV+: now also J1.29 (Pin_29), C2.1
- net LV-: now also C2.2
- new net I_hv_+: J1.12 (Pin_12)
- new net I_hv_-: J1.6 (Pin_6)
- new net I_lv_+: J1.32 (Pin_32)
- new net I_lv_-: J1.30 (Pin_30)
Other:
- note added: "Power flow"
- note removed: "12V power"
- moved on the sheet: C10, C4, C8, C9
